File: stm32_plug'n'play/stm32_plug'n'play.kicad_sch (KiCad schematic)
At the start: 48 parts, among them J1 Screw_Terminal_01x02, J2 USB_B_Micro, SW1 SW_SPDT, U1 STM32F302C8Tx, U2 AMS1117-3.3, U3 BMP388, U4 MPU-6050, U5 TMP112, Y1 X322516MLB4SI

Commit message: Add files via upload
Parts:
- D3, D4, D5: footprint LED_SMD:LED_1210_3225Metric -> LED_SMD:LED_0805_2012Metric
- R1, R10, R11, R2, R3, R4, R5, R6, R7, R8, R9: footprint Resistor_SMD:R_0603_1608Metric -> Resistor_SMD:R_0402_1005Metric
Changed lines of the file:
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@@
       (effects (font (size 1.27 1.27)) hide)
     )
-    (property "Footprint" "Resistor_SMD:R_0603_1608Metric" (id 2) (at 73.025 175.895 0)
+    (property "Footprint" "Resistor_SMD:R_0402_1005Metric" (id 2) (at 73.025 175.895 0)
       (effects (font (size 1.27 1.27)) hide)
     )
@@
       (effects (font (size 1.27 1.27)) (justify right))
     )
-    (property "Footprint" "LED_SMD:LED_1210_3225Metric" (id 2) (at 73.025 181.61 90)
+    (property "Footprint" "LED_SMD:LED_0805_2012Metric" (id 2) (at 73.025 181.61 90)
       (effects (font (size 1.27 1.27)) hide)
     )
@@
       (effects (font (size 1.27 1.27)) hide)
     )
-    (property "Footprint" "Resistor_SMD:R_0603_1608Metric" (id 2) (at 90.805 27.94 0)
+    (property "Footprint" "Resistor_SMD:R_0402_1005Metric" (id 2) (at 90.805 27.94 0)
       (effects (font (size 1.27 1.27)) hide)
     )
@@
     (property "Reference" "R4" (id 0) (at 78.74 83.82 90))
     (property "Value" "330" (id 1) (at 78.74 88.265 90))
-    (property "Footprint" "Resistor_SMD:R_0603_1608Metric" (id 2) (at 78.74 85.725 0)
+    (property "Footprint" "Resistor_SMD:R_0402_1005Metric" (id 2) (at 78.74 85.725 0)
       (effects (font (size 1.27 1.27)) hide)
     )
@@
     (property "Reference" "R3" (id 0) (at 78.74 77.2945 90))
     (property "Value" "330" (id 1) (at 78.74 81.915 90))
-    (property "Footprint" "Resistor_SMD:R_0603_1608Metric" (id 2) (at 78.74 79.375 0)
+    (property "Footprint" "Resistor_SMD:R_0402_1005Metric" (id 2) (at 78.74 79.375 0)
       (effects (font (size 1.27 1.27)) hide)
     )
@@
       (effects (font (size 1.27 1.27)) (justify left))
     )
-    (property "Footprint" "Resistor_SMD:R_0603_1608Metric" (id 2) (at 251.46 86.995 0)
+    (property "Footprint" "Resistor_SMD:R_0402_1005Metric" (id 2) (at 251.46 86.995 0)
       (effects (font (size 1.27 1.27)) hide)
     )
@@
       (effects (font (size 1.27 1.27)) hide)
     )
-    (property "Footprint" "LED_SMD:LED_1210_3225Metric" (id 2) (at 85.725 85.725 90)
+    (property "Footprint" "LED_SMD:LED_0805_2012Metric" (id 2) (at 85.725 85.725 90)
       (effects (font (size 1.27 1.27)) hide)
     )
@@
       (effects (font (size 1.27 1.27)) (justify left))
     )
-    (property "Footprint" "Resistor_SMD:R_0603_1608Metric" (id 2) (at 233.68 129.54 0)
+    (property "Footprint" "Resistor_SMD:R_0402_1005Metric" (id 2) (at 233.68 129.54 0)
       (effects (font (size 1.27 1.27)) hide)
     )
@@
       (effects (font (size 1.27 1.27)) (justify left))
     )
-    (property "Footprint" "Resistor_SMD:R_0603_1608Metric" (id 2) (at 228.6 129.54 0)
+    (property "Footprint" "Resistor_SMD:R_0402_1005Metric" (id 2) (at 228.6 129.54 0)
       (effects (font (size 1.27 1.27)) hide)
     )
@@
       (effects (font (size 1.27 1.27)) (justify right) hide)
     )
-    (property "Footprint" "Resistor_SMD:R_0603_1608Metric" (id 2) (at 75.565 102.235 0)
+    (property "Footprint" "Resistor_SMD:R_0402_1005Metric" (id 2) (at 75.565 102.235 0)
       (effects (font (size 1.27 1.27)) hide)
     )
@@
       (effects (font (size 1.27 1.27)) hide)
     )
-    (property "Footprint" "LED_SMD:LED_1210_3225Metric" (id 2) (at 85.725 79.375 90)
+    (property "Footprint" "LED_SMD:LED_0805_2012Metric" (id 2) (at 85.725 79.375 90)
       (effects (font (size 1.27 1.27)) hide)
     )
@@
       (effects (font (size 1.27 1.27)) hide)
     )
-    (property "Footprint" "Resistor_SMD:R_0603_1608Metric" (id 2) (at 258.445 33.02 0)
+    (property "Footprint" "Resistor_SMD:R_0402_1005Metric" (id 2) (at 258.445 33.02 0)
       (effects (font (size 1.27 1.27)) hide)
     )
@@
       (effects (font (size 1.27 1.27)) (justify left))
     )
-    (property "Footprint" "Resistor_SMD:R_0603_1608Metric" (id 2) (at 241.3 86.995 0)
+    (property "Footprint" "Resistor_SMD:R_0402_1005Metric" (id 2) (at 241.3 86.995 0)
       (effects (font (size 1.27 1.27)) hide)
     )
@@
       (effects (font (size 1.27 1.27)) (justify left))
     )
-    (property "Footprint" "Resistor_SMD:R_0603_1608Metric" (id 2) (at 246.38 86.995 0)
+    (property "Footprint" "Resistor_SMD:R_0402_1005Metric" (id 2) (at 246.38 86.995 0)
       (effects (font (size 1.27 1.27)) hide)
     )
@@
     )
     (path "/34006235-2cfc-4273-a2ba-1d67db1e08b2"
-      (reference "D3") (unit 1) (value "LED_Green") (footprint "LED_SMD:LED_1210_3225Metric")
+      (reference "D3") (unit 1) (value "LED_Green") (footprint "LED_SMD:LED_0805_2012Metric")
     )
     (path "/d4da85f7-e51a-4516-a132-54ed1dab8445"
-      (reference "D4") (unit 1) (value "LED_Blue") (footprint "LED_SMD:LED_1210_3225Metric")
+      (reference "D4") (unit 1) (value "LED_Blue") (footprint "LED_SMD:LED_0805_2012Metric")
     )
     (path "/963b190e-28f1-49fb-83ae-04bb5c03ea41"
-      (reference "D5") (unit 1) (value "LED_Red") (footprint "LED_SMD:LED_1210_3225Metric")
+      (reference "D5") (unit 1) (value "LED_Red") (footprint "LED_SMD:LED_0805_2012Metric")
     )
     (path "/23daa4da-8a9b-4322-8490-40d7db781117"
@@
     )
     (path "/23f7c4b9-b044-4936-9e74-e88336bdb924"
-      (reference "R1") (unit 1) (value "330") (footprint "Resistor_SMD:R_0603_1608Metric")
+      (reference "R1") (unit 1) (value "330") (footprint "Resistor_SMD:R_0402_1005Metric")
     )
     (path "/cbd2d2d6-45c1-48d1-824b-d821332953ab"
-      (reference "R2") (unit 1) (value "1.5k") (footprint "Resistor_SMD:R_0603_1608Metric")
+      (reference "R2") (unit 1) (value "1.5k") (footprint "Resistor_SMD:R_0402_1005Metric")
     )
     (path "/6120253c-1f2b-4282-8a17-22042c76cef8"
-      (reference "R3") (unit 1) (value "330") (footprint "Resistor_SMD:R_0603_1608Metric")
+      (reference "R3") (unit 1) (value "330") (footprint "Resistor_SMD:R_0402_1005Metric")
     )
     (path "/5c403879-1e42-47bd-adcf-a43333800b85"
-      (reference "R4") (unit 1) (value "330") (footprint "Resistor_SMD:R_0603_1608Metric")
+      (reference "R4") (unit 1) (value "330") (footprint "Resistor_SMD:R_0402_1005Metric")
     )
     (path "/46580b33-dd5a-4ec3-bdd9-d719d377ad71"
-      (reference "R5") (unit 1) (value "47") (footprint "Resistor_SMD:R_0603_1608Metric")
+      (reference "R5") (unit 1) (value "47") (footprint "Resistor_SMD:R_0402_1005Metric")
     )
     (path "/c2ef9bcd-6dac-4a06-94a7-eed2e9d97ccf"
-      (reference "R6") (unit 1) (value "4.7k") (footprint "Resistor_SMD:R_0603_1608Metric")
+      (reference "R6") (unit 1) (value "4.7k") (footprint "Resistor_SMD:R_0402_1005Metric")
     )
     (path "/c22f4e91-863c-462a-ac49-1b69efe59912"
-      (reference "R7") (unit 1) (value "4.7k") (footprint "Resistor_SMD:R_0603_1608Metric")
+      (reference "R7") (unit 1) (value "4.7k") (footprint "Resistor_SMD:R_0402_1005Metric")
     )
     (path "/e12bfad0-8d05-4e76-aaec-ab3cda8b5b3d"
-      (reference "R8") (unit 1) (value "4.7k") (footprint "Resistor_SMD:R_0603_1608Metric")
+      (reference "R8") (unit 1) (value "4.7k") (footprint "Resistor_SMD:R_0402_1005Metric")
     )
     (path "/fa0167fd-4124-4087-8c8d-46ef9fe29193"
-      (reference "R9") (unit 1) (value "4.7k") (footprint "Resistor_SMD:R_0603_1608Metric")
+      (reference "R9") (unit 1) (value "4.7k") (footprint "Resistor_SMD:R_0402_1005Metric")
     )
     (path "/71bb6a83-ed45-4d29-96a6-d41f48385263"
-      (reference "R10") (unit 1) (value "4.7k") (footprint "Resistor_SMD:R_0603_1608Metric")
+      (reference "R10") (unit 1) (value "4.7k") (footprint "Resistor_SMD:R_0402_1005Metric")
     )
     (path "/de408512-0845-4302-b8c2-09a96f52358b"
-      (reference "R11") (unit 1) (value "10k") (footprint "Resistor_SMD:R_0603_1608Metric")
+      (reference "R11") (unit 1) (value "10k") (footprint "Resistor_SMD:R_0402_1005Metric")
     )
     (path "/66c2b40c-008b-4c4e-acb9-a610ad8b78e1"
